File: PCBs/E-Latch/E-Latch_Type3/E-Latch.sch (KiCad schematic (older format))
At the start: 17 parts, among them J3 MOTOR, K1 G5LE-1, K2 G5LE-1, K3 G5LE-1, U1 LM1117-3.3

Commit message: Update device
Parts:
- gave numbers to parts that had none: 2
Changed lines of the file:
@@
 $EndBitmap
 $Comp
-L Connector:Conn_01x02_Male J?
+L Connector:Conn_01x02_Male J2
 U 1 1 603E2C87
 P 2400 4300
-F 0 "J?" H 2508 4481 50  0000 C CNN
+F 0 "J2" H 2508 4481 50  0000 C CNN
 F 1 "SIG" H 2508 4390 50  0000 C CNN
 F 2 "Connector_Phoenix_MSTB:PhoenixContact_MSTBVA_2,5_2-G-5,08_1x02_P5.08mm_Vertical" H 2400 4300 50  0001 C CNN
@@
 $EndComp
 $Comp
-L Connector:Conn_01x02_Male J?
+L Connector:Conn_01x02_Male J1
 U 1 1 603E3D87
 P 2400 1900
-F 0 "J?" H 2508 2081 50  0000 C CNN
+F 0 "J1" H 2508 2081 50  0000 C CNN
 F 1 "POWER" H 2508 1990 50  0000 C CNN
 F 2 "Connector_Phoenix_MSTB:PhoenixContact_MSTBVA_2,5_2-G-5,08_1x02_P5.08mm_Vertical" H 2400 1900 50  0001 C CNN
@@
 	2600 1900 4150 1900
 $Comp
-L power:GND #PWR?
+L power:GND #PWR08
 U 1 1 603EB349
 P 2750 4550
-F 0 "#PWR?" H 2750 4300 50  0001 C CNN
+F 0 "#PWR08" H 2750 4300 50  0001 C CNN
 F 1 "GND" H 2755 4377 50  0000 C CNN
 F 2 "" H 2750 4550 50  0001 C CNN

Commit message: Rebuild Type 3 of E-Latch
Parts:
- C1, C5: symbol Device:C -> E-Latch-rescue:C-Device
- C2, C3, C4, C6, C7: symbol Device:CP -> E-Latch-rescue:CP-Device
- D1, D2, D3: symbol Diode:1N4007 -> E-Latch-rescue:1N4007-Diode
- J1, J2, J3: symbol Connector:Conn_01x02_Male -> E-Latch-rescue:Conn_01x02_Male-Connector
- K1, K2, K3: symbol Relay:G5LE-1 -> E-Latch-rescue:G5LE-1-Relay
- U1: symbol Regulator_Linear:LM1117-3.3 -> E-Latch-rescue:LM1117-3.3-Regulator_Linear
Changed lines of the file:
@@
 $EndDescr
 $Comp
-L Device:C C1
+L E-Latch-rescue:C-Device C1
 U 1 1 5DE7C345
 P 4150 2250
@@
 $EndComp
 $Comp
-L Device:CP C2
+L E-Latch-rescue:CP-Device C2
 U 1 1 5DE7CDC8
 P 4650 2250
@@
 $EndComp
 $Comp
-L Regulator_Linear:LM1117-3.3 U1
+L E-Latch-rescue:LM1117-3.3-Regulator_Linear U1
 U 1 1 5DE7D658
 P 5350 1900
@@
 	4150 1900 4650 1900
 $Comp
-L power:GND #PWR01
+L E-Latch-rescue:GND-power #PWR01
 U 1 1 5DE7ED8C
 P 3800 2550
@@
 Connection ~ 4650 2500
 $Comp
-L Device:C C5
+L E-Latch-rescue:C-Device C5
 U 1 1 5DE80683
 P 5950 2250
@@
 $EndComp
 $Comp
-L Device:CP C6
+L E-Latch-rescue:CP-Device C6
 U 1 1 5DE80F8A
 P 6500 2250
@@
 Connection ~ 5950 2500
 $Comp
-L power:+3.3V #PWR05
+L E-Latch-rescue:+3.3V-power #PWR05
 U 1 1 5DE82058
 P 6500 1800
@@
 Connection ~ 6500 1900
 $Comp
-L power:+24V #PWR02
+L E-Latch-rescue:+24V-power #PWR02
 U 1 1 5DE82A2C
 P 4150 1800
@@
 	4150 1900 4150 1800
 $Comp
-L Device:CP C4
+L E-Latch-rescue:CP-Device C4
 U 1 1 5DE8391C
 P 5300 5150
@@
 $EndComp
 $Comp
-L Diode:1N4007 D2
+L E-Latch-rescue:1N4007-Diode D2
 U 1 1 5DE83C79
 P 6350 5900
@@
 $EndComp
 $Comp
-L Relay:G5LE-1 K1
+L E-Latch-rescue:G5LE-1-Relay K1
 U 1 1 5DE7CD07
 P 4350 4500
@@
 $EndComp
 $Comp
-L Relay:G5LE-1 K2
+L E-Latch-rescue:G5LE-1-Relay K2
 U 1 1 5DE7E52A
 P 6900 4200
@@
 $EndComp
 $Comp
-L Relay:G5LE-1 K3
+L E-Latch-rescue:G5LE-1-Relay K3
 U 1 1 5DE7F895
 P 6900 5200
@@
 $EndComp
 $Comp
-L Connector:Conn_01x02_Male J3
+L E-Latch-rescue:Conn_01x02_Male-Connector J3
 U 1 1 5DE80427
 P 9150 4700
@@
 	7200 3800 7200 3900
 $Comp
-L power:+3.3V #PWR07
+L E-Latch-rescue:+3.3V-power #PWR07
 U 1 1 5DE860EF
 P 7800 3600
@@
 $EndComp
 $Comp
-L power:GND #PWR06
+L E-Latch-rescue:GND-power #PWR06
 U 1 1 5DE86AC5
 P 7700 4900
@@
 Connection ~ 7800 3800
 $Comp
-L Device:CP C7
+L E-Latch-rescue:CP-Device C7
 U 1 1 5DE89D31
 P 8200 5100
@@
 	8200 5600 8700 5600
 $Comp
-L Diode:1N4007 D1
+L E-Latch-rescue:1N4007-Diode D1
 U 1 1 5DE8E6EB
 P 6300 3500
@@
 	6700 4900 6700 4700
 $Comp
-L Device:CP C3
+L E-Latch-rescue:CP-Device C3
 U 1 1 5DE92110
 P 5300 4250
@@
 	5900 5900 6200 5900
 $Comp
-L power:+24V #PWR03
+L E-Latch-rescue:+24V-power #PWR03
 U 1 1 5DEA5349
 P 5300 3350
@@
 	5300 3350 5300 3700
 $Comp
-L power:GND #PWR04
+L E-Latch-rescue:GND-power #PWR04
 U 1 1 5DEA6EA5
 P 5300 5650
@@
 Connection ~ 5900 5900
 $Comp
-L Diode:1N4007 D3
+L E-Latch-rescue:1N4007-Diode D3
 U 1 1 5EEB4CE7
 P 4350 3700
@@
 $EndBitmap
 $Comp
-L Connector:Conn_01x02_Male J2
+L E-Latch-rescue:Conn_01x02_Male-Connector J2
 U 1 1 603E2C87
 P 2400 4300
@@
 $EndComp
 $Comp
-L Connector:Conn_01x02_Male J1
+L E-Latch-rescue:Conn_01x02_Male-Connector J1
 U 1 1 603E3D87
 P 2400 1900
@@
 	2600 1900 4150 1900
 $Comp
-L power:GND #PWR08
+L E-Latch-rescue:GND-power #PWR08
 U 1 1 603EB349
 P 2750 4550
