File: PCBs/Lamps/Lamps_Type3/Lamls_Type3.sch (KiCad schematic (older format))
At the start: 35 parts, among them J1 IN, J2 POWER, J3 LAMP2, J4 LAMP3, J5 LAMP4, J6 LAMP1, J7 LAMP5, J8 LAMP6, Q1 2N2222, Q2 2N2222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

Commit message: Add fiducials for machine ready work
Parts:
- gave numbers to parts that had none: 3
Changed lines of the file:
@@
 Connection ~ 1450 6200
 $Comp
-L Mechanical:Fiducial FID?
+L Mechanical:Fiducial FID1
 U 1 1 6124D72B
 P 5550 7550
-F 0 "FID?" H 5635 7596 50  0000 L CNN
+F 0 "FID1" H 5635 7596 50  0000 L CNN
 F 1 "Fiducial" H 5635 7505 50  0000 L CNN
 F 2 "Fiducial:Fiducial_0.5mm_Mask1.5mm" H 5550 7550 50  0001 C CNN
@@
 $EndComp
 $Comp
-L Mechanical:Fiducial FID?
+L Mechanical:Fiducial FID2
 U 1 1 6124DC8B
 P 6050 7550
-F 0 "FID?" H 6135 7596 50  0000 L CNN
+F 0 "FID2" H 6135 7596 50  0000 L CNN
 F 1 "Fiducial" H 6135 7505 50  0000 L CNN
 F 2 "Fiducial:Fiducial_0.5mm_Mask1.5mm" H 6050 7550 50  0001 C CNN
@@
 $EndComp
 $Comp
-L Mechanical:Fiducial FID?
+L Mechanical:Fiducial FID3
 U 1 1 6124E0C8
 P 6550 7550
-F 0 "FID?" H 6635 7596 50  0000 L CNN
+F 0 "FID3" H 6635 7596 50  0000 L CNN
 F 1 "Fiducial" H 6635 7505 50  0000 L CNN
 F 2 "Fiducial:Fiducial_0.5mm_Mask1.5mm" H 6550 7550 50  0001 C CNN
