File: PCBs/Lamps/LDR-0-10V/LDR-0-10V.kicad_pcb (KiCad board)
At the start: 2 copper layers, 43.2 x 43.2 mm, 10 parts, among them J1 CON, U1 LM358

Commit message: Update LDR-0-10V
Parts:
- moved RV1 11.7 mm to (128.9, 94.8), turned to 270 degrees
Connections:
- RV1 pad 2: GND -> Net-(C2-Pad1)
Routing:
- net Net-(C2-Pad1): track 27.7 -> 44.6 mm
- net AO: track 41.9 -> 36.9 mm
Other:
- board text added: "ZTM-LS-V1"
